Commit message: my_robot.xacro file repaired

File: catkin_ws/src/my_robot/urdf/my_robot.xacro (robot description, xacro)
@@ -1,9 +1,7 @@
 <?xml version='1.0'?>
 <robot name="my_robot" xmlns:xacro="http://www.ros.org/wiki/xacro">
-  <xacro:include filename="$(find my_robot)/urdf/my_robot.gazebo" />
-  <!-- links -->
   <link name="robot_footprint"></link>
-   <link name='chassis'>
-    <pose>0 0 0.1 0 0 0</pose>
+  <link name='chassis'>
+    <pose>0 0 0.075 0 0 0</pose>
     <inertial>
       <mass value="15.0"/>
@@ -15,8 +13,8 @@
       />
     </inertial>
-    <collision name='collision'>
+    <collision name='chassis_collision'>
       <origin xyz="0 0 0" rpy=" 0 0 0"/>
       <geometry>
-        <box size=".4 .2 .1"/>
+        <box size=".4 .2 .05"/>
       </geometry>
     </collision>
@@ -24,9 +22,9 @@
       <origin xyz="0 0 0" rpy=" 0 0 0"/>
       <geometry>
-        <box size=".4 .2 .1"/>
+        <box size=".4 .2 .05"/>
       </geometry>
     </visual>
     <collision name='back_caster_collision'>
-      <origin xyz="-0.15 0 -0.05" rpy=" 0 0 0"/>
+      <origin xyz="-0.15 0 -0.025" rpy=" 0 0 0"/>
       <geometry>
         <sphere radius="0.0499"/>
@@ -34,11 +32,11 @@
     </collision>
     <visual name='back_caster_visual'>
-      <origin xyz="-0.15 0 -0.05" rpy=" 0 0 0"/>
+      <origin xyz="-0.15 0 -0.025" rpy=" 0 0 0"/>
       <geometry>
         <sphere radius="0.05"/>
       </geometry>
     </visual>
-    <collision name='front_caster_collision'>
-      <origin xyz="0.15 0 -0.05" rpy=" 0 0 0"/>
+   <collision name='front_caster_collision'>
+      <origin xyz="0.15 0 -0.025" rpy=" 0 0 0"/>
       <geometry>
         <sphere radius="0.0499"/>
@@ -46,5 +44,5 @@
     </collision>
     <visual name='front_caster_visual'>
-      <origin xyz="0.15 0 -0.05" rpy=" 0 0 0"/>
+      <origin xyz="0.15 0 -0.025" rpy=" 0 0 0"/>
       <geometry>
         <sphere radius="0.05"/>
@@ -65,5 +63,5 @@
       <origin xyz="0.0 0 0" rpy="0 1.5707 1.5707"/>
       <geometry>
-        <cylinder radius="0.1" length="0.05"/>
+        <cylinder radius="0.075" length="0.08"/>
       </geometry>
     </collision>
@@ -71,5 +69,5 @@
       <origin xyz="0.0 0 0" rpy="0 1.5707 1.5707"/>
       <geometry>
-        <cylinder radius="0.1" length="0.05"/>
+        <cylinder radius="0.075" length="0.08"/>
       </geometry>
     </visual>
@@ -85,14 +83,14 @@
       />
     </inertial>
-    <collision name='left_wheel_collision'>
+    <collision name='right_wheel_collision'>
       <origin xyz="0.0 0 0" rpy="0 1.5707 1.5707"/>
       <geometry>
-        <cylinder radius="0.1" length="0.05"/>
+        <cylinder radius="0.075" length="0.08"/>
       </geometry>
     </collision>
-    <visual name='left_wheel_visual'>
+    <visual name='right_wheel_visual'>
       <origin xyz="0.0 0 0" rpy="0 1.5707 1.5707"/>
       <geometry>
-        <cylinder radius="0.1" length="0.05"/>
+        <cylinder radius="0.075" length="0.08"/>
       </geometry>
     </visual>
@@ -111,5 +109,5 @@
       <origin xyz="0 0 0" rpy=" 0 0 0"/>
       <geometry>
-        <box size=".05 .05 .05"/>
+        <box size=".025 .08 .05"/>
       </geometry>
     </collision>
@@ -117,5 +115,5 @@
       <origin xyz="0 0 0" rpy=" 0 0 0"/>
       <geometry>
-        <box size=".05 .05 .05"/>
+        <box size=".025 .08 .05"/>
       </geometry>
     </visual>
@@ -145,5 +143,5 @@
   </link>
   <!-- joints -->
- <joint name="robot_footprint_joint" type="fixed">
+  <joint name="robot_footprint_joint" type="fixed">
     <origin xyz="0 0 0" rpy="0 0 0" />
     <parent link="robot_footprint"/>
@@ -151,5 +149,5 @@
   </joint>
   <joint name="left_wheel_hinge" type="continuous" >
-    <origin xyz="0 0.15 0" rpy="0 0 0"/>
+    <origin xyz="0.125 0.15 0" rpy="0 0 0"/>
     <child link="left_wheel"/>
     <parent link="chassis"/>
@@ -159,5 +157,5 @@
   </joint>
   <joint name="right_wheel_hinge" type="continuous" >
-    <origin xyz="0 -0.15 0" rpy="0 0 0"/>
+    <origin xyz="0.125 -0.15 0" rpy="0 0 0"/>
     <child link="right_wheel"/>
     <parent link="chassis"/>
@@ -167,5 +165,5 @@
   </joint>
   <joint name="camera_joint" type="fixed">
-    <origin xyz="0.2 0 0" rpy="0 0 0" />
+    <origin xyz="0.2125 0 0" rpy="0 0 0" />
     <parent link="chassis"/>
     <child link="camera" />
@@ -173,5 +171,5 @@
   </joint>
   <joint name="hokuyo_joint" type="fixed">
-    <origin xyz=".15 0 .1" rpy="0 0 0" />
+    <origin xyz=".15 0 .075" rpy="0 0 0" />
     <parent link="chassis"/>
     <child link="hokuyo" />
@@ -180,5 +178,5 @@
   <!-- colors -->
   <gazebo reference="left_wheel">
-    <material>Gazebo/Green</material>
+    <material>Gazebo/Red</material>
   </gazebo>
   <gazebo reference="right_wheel">
@@ -186,8 +184,8 @@
   </gazebo>
   <gazebo reference="chassis">
-    <material>Gazebo/Blue</material>
+    <material>Gazebo/Orange</material>
   </gazebo>
   <gazebo reference="camera">
-    <material>Gazebo/Red</material>
+    <material>Gazebo/Yellow</material>
   </gazebo>
 </robot>

Commit message: updated program and robot

File: catkin_ws/src/my_robot/urdf/my_robot.xacro (robot description, xacro)
@@ -1,9 +1,10 @@
 <?xml version='1.0'?>
 <robot name="my_robot" xmlns:xacro="http://www.ros.org/wiki/xacro">
+  <xacro:include filename="$(find my_robot)/urdf/my_robot.gazebo" />
   <link name="robot_footprint"></link>
   <link name='chassis'>
     <pose>0 0 0.075 0 0 0</pose>
     <inertial>
-      <mass value="15.0"/>
+      <mass value="10.0"/>
       <origin xyz="0.0 0 0" rpy=" 0 0 0"/>
       <inertia
@@ -16,5 +17,5 @@
       <origin xyz="0 0 0" rpy=" 0 0 0"/>
       <geometry>
-        <box size=".4 .2 .05"/>
+        <box size=".3 .2 .05"/>
       </geometry>
     </collision>
@@ -22,9 +23,9 @@
       <origin xyz="0 0 0" rpy=" 0 0 0"/>
       <geometry>
-        <box size=".4 .2 .05"/>
+        <box size=".3 .2 .05"/>
       </geometry>
     </visual>
     <collision name='back_caster_collision'>
-      <origin xyz="-0.15 0 -0.025" rpy=" 0 0 0"/>
+      <origin xyz="-0.10 0 -0.025" rpy=" 0 0 0"/>
       <geometry>
         <sphere radius="0.0499"/>
@@ -32,5 +33,5 @@
     </collision>
     <visual name='back_caster_visual'>
-      <origin xyz="-0.15 0 -0.025" rpy=" 0 0 0"/>
+      <origin xyz="-0.10 0 -0.025" rpy=" 0 0 0"/>
       <geometry>
         <sphere radius="0.05"/>
@@ -38,5 +39,5 @@
     </visual>
    <collision name='front_caster_collision'>
-      <origin xyz="0.15 0 -0.025" rpy=" 0 0 0"/>
+      <origin xyz="0.10 0 -0.025" rpy=" 0 0 0"/>
       <geometry>
         <sphere radius="0.0499"/>
@@ -44,5 +45,5 @@
     </collision>
     <visual name='front_caster_visual'>
-      <origin xyz="0.15 0 -0.025" rpy=" 0 0 0"/>
+      <origin xyz="0.10 0 -0.025" rpy=" 0 0 0"/>
       <geometry>
         <sphere radius="0.05"/>
@@ -149,5 +150,5 @@
   </joint>
   <joint name="left_wheel_hinge" type="continuous" >
-    <origin xyz="0.125 0.15 0" rpy="0 0 0"/>
+    <origin xyz="0.075 0.15 0" rpy="0 0 0"/>
     <child link="left_wheel"/>
     <parent link="chassis"/>
@@ -157,5 +158,5 @@
   </joint>
   <joint name="right_wheel_hinge" type="continuous" >
-    <origin xyz="0.125 -0.15 0" rpy="0 0 0"/>
+    <origin xyz="0.075 -0.15 0" rpy="0 0 0"/>
     <child link="right_wheel"/>
     <parent link="chassis"/>
@@ -165,5 +166,5 @@
   </joint>
   <joint name="camera_joint" type="fixed">
-    <origin xyz="0.2125 0 0" rpy="0 0 0" />
+    <origin xyz="0.1625 0 0" rpy="0 0 0" />
     <parent link="chassis"/>
     <child link="camera" />
@@ -171,5 +172,5 @@
   </joint>
   <joint name="hokuyo_joint" type="fixed">
-    <origin xyz=".15 0 .075" rpy="0 0 0" />
+    <origin xyz=".10 0 .075" rpy="0 0 0" />
     <parent link="chassis"/>
     <child link="hokuyo" />

Commit message: fix: correct the robot moving too slow changes made: -increased robot linear and angular speeds;  - modified robot xacro with thinner wheels and more central position.

File: catkin_ws/src/my_robot/urdf/my_robot.xacro (robot description, xacro)
@@ -64,5 +64,5 @@
       <origin xyz="0.0 0 0" rpy="0 1.5707 1.5707"/>
       <geometry>
-        <cylinder radius="0.075" length="0.08"/>
+        <cylinder radius="0.075" length="0.04"/>
       </geometry>
     </collision>
@@ -70,5 +70,5 @@
       <origin xyz="0.0 0 0" rpy="0 1.5707 1.5707"/>
       <geometry>
-        <cylinder radius="0.075" length="0.08"/>
+        <cylinder radius="0.075" length="0.04"/>
       </geometry>
     </visual>
@@ -87,5 +87,5 @@
       <origin xyz="0.0 0 0" rpy="0 1.5707 1.5707"/>
       <geometry>
-        <cylinder radius="0.075" length="0.08"/>
+        <cylinder radius="0.075" length="0.04"/>
       </geometry>
     </collision>
@@ -93,5 +93,5 @@
       <origin xyz="0.0 0 0" rpy="0 1.5707 1.5707"/>
       <geometry>
-        <cylinder radius="0.075" length="0.08"/>
+        <cylinder radius="0.075" length="0.04"/>
       </geometry>
     </visual>
@@ -150,5 +150,5 @@
   </joint>
   <joint name="left_wheel_hinge" type="continuous" >
-    <origin xyz="0.075 0.15 0" rpy="0 0 0"/>
+    <origin xyz="0.05 0.125 0" rpy="0 0 0"/>
     <child link="left_wheel"/>
     <parent link="chassis"/>
@@ -158,5 +158,5 @@
   </joint>
   <joint name="right_wheel_hinge" type="continuous" >
-    <origin xyz="0.075 -0.15 0" rpy="0 0 0"/>
+    <origin xyz="0.05 -0.125 0" rpy="0 0 0"/>
     <child link="right_wheel"/>
     <parent link="chassis"/>

Commit message: bug: corrected robot inestability
Following recommendation from mentor (see question: https://knowledge.udacity.com/questions/282631
robot weights, casterballs and geometry was changed to make it more stable.
the robot drives more stable, (although it still drifts a bit). And also can localize itself better.
TODO: improve amcl parameters to improve localization.

File: catkin_ws/src/my_robot/urdf/my_robot.xacro (robot description, xacro)
@@ -6,10 +6,10 @@
     <pose>0 0 0.075 0 0 0</pose>
     <inertial>
-      <mass value="10.0"/>
+      <mass value="20.0"/>
       <origin xyz="0.0 0 0" rpy=" 0 0 0"/>
       <inertia
-          ixx="0.1" ixy="0" ixz="0"
-          iyy="0.1" iyz="0"
-          izz="0.1"
+          ixx="0.08" ixy="0" ixz="0"
+          iyy="0.15" iyz="0"
+          izz="0.22"
       />
     </inertial>
@@ -27,25 +27,25 @@
     </visual>
     <collision name='back_caster_collision'>
-      <origin xyz="-0.10 0 -0.025" rpy=" 0 0 0"/>
+      <origin xyz="-0.10 0 -0.055" rpy=" 0 0 0"/>
       <geometry>
-        <sphere radius="0.0499"/>
+        <sphere radius="0.0199"/>
       </geometry>
     </collision>
     <visual name='back_caster_visual'>
-      <origin xyz="-0.10 0 -0.025" rpy=" 0 0 0"/>
+      <origin xyz="-0.10 0 -0.055" rpy=" 0 0 0"/>
       <geometry>
-        <sphere radius="0.05"/>
+        <sphere radius="0.020"/>
       </geometry>
     </visual>
-   <collision name='front_caster_collision'>
-      <origin xyz="0.10 0 -0.025" rpy=" 0 0 0"/>
+    <collision name='front_caster_collision'>
+      <origin xyz="0.10 0 -0.055" rpy=" 0 0 0"/>
       <geometry>
-        <sphere radius="0.0499"/>
+        <sphere radius="0.0199"/>
       </geometry>
     </collision>
     <visual name='front_caster_visual'>
-      <origin xyz="0.10 0 -0.025" rpy=" 0 0 0"/>
+      <origin xyz="0.10 0 -0.055" rpy=" 0 0 0"/>
       <geometry>
-        <sphere radius="0.05"/>
+        <sphere radius="0.020"/>
       </geometry>
     </visual>
@@ -53,14 +53,13 @@
   <link name='left_wheel'>
     <inertial>
-      <mass value="5.0"/>
-      <origin xyz="0.0 0 0" rpy="0 1.5707 1.5707"/>
+      <mass value="10.0"/>
       <inertia
-          ixx="0.1" ixy="0" ixz="0"
-          iyy="0.1" iyz="0"
-          izz="0.1"
+          ixx="0.015" ixy="0" ixz="0"
+          iyy="0.015" iyz="0"
+          izz="0.030"
       />
     </inertial>
     <collision name='left_wheel_collision'>
-      <origin xyz="0.0 0 0" rpy="0 1.5707 1.5707"/>
+      <origin xyz="0.0 0 0" rpy="1.5707 0 0"/>
       <geometry>
         <cylinder radius="0.075" length="0.04"/>
@@ -68,5 +67,5 @@
     </collision>
     <visual name='left_wheel_visual'>
-      <origin xyz="0.0 0 0" rpy="0 1.5707 1.5707"/>
+      <origin xyz="0.0 0 0" rpy="1.5707 0  0"/>
       <geometry>
         <cylinder radius="0.075" length="0.04"/>
@@ -75,15 +74,14 @@
   </link>
   <link name='right_wheel'>
-    <inertial>
-      <mass value="5.0"/>
-      <origin xyz="0.0 0 0" rpy="0 1.5707 1.5707"/>
+     <inertial>
+      <mass value="10.0"/>
       <inertia
-          ixx="0.1" ixy="0" ixz="0"
-          iyy="0.1" iyz="0"
-          izz="0.1"
+          ixx="0.015" ixy="0" ixz="0"
+          iyy="0.015" iyz="0"
+          izz="0.030"
       />
     </inertial>
     <collision name='right_wheel_collision'>
-      <origin xyz="0.0 0 0" rpy="0 1.5707 1.5707"/>
+      <origin xyz="0.0 0 0" rpy="1.5707 0 0"/>
       <geometry>
         <cylinder radius="0.075" length="0.04"/>
@@ -91,5 +89,5 @@
     </collision>
     <visual name='right_wheel_visual'>
-      <origin xyz="0.0 0 0" rpy="0 1.5707 1.5707"/>
+      <origin xyz="0.0 0 0" rpy="1.5707 0  0"/>
       <geometry>
         <cylinder radius="0.075" length="0.04"/>
@@ -148,7 +146,8 @@
     <parent link="robot_footprint"/>
     <child link="chassis" />
+    <dynamics friction="0.0"/>
   </joint>
   <joint name="left_wheel_hinge" type="continuous" >
-    <origin xyz="0.05 0.125 0" rpy="0 0 0"/>
+    <origin xyz="0.00 0.125 0" rpy="0 0 0"/>
     <child link="left_wheel"/>
     <parent link="chassis"/>
@@ -158,5 +157,5 @@
   </joint>
   <joint name="right_wheel_hinge" type="continuous" >
-    <origin xyz="0.05 -0.125 0" rpy="0 0 0"/>
+    <origin xyz="0.00 -0.125 0" rpy="0 0 0"/>
     <child link="right_wheel"/>
     <parent link="chassis"/>
